Commit message: set inertial for gripper find pad

File: kube_bullet/robots/robot_assets/ur10e_cell/ur10e_cell.urdf (robot description, URDF)
Before this commit: robot ur10e_cell, 38 links, 37 joints
Links:
- link left_inner_finger_pad: mass None -> 0.08
- link right_inner_finger_pad: mass None -> 0.08
